File: hardware/box-v1/kicad/mcu.kicad_sch (KiCad schematic)
At the start: 24 parts, among them U301 CH32V305RBT6, X301 8MHz

Commit message: hardware/box-v1 in English, with an order package
- Everything in hardware/box-v1 is English: netlist.py, the generators,
  the checks, the README, and the regenerated KiCad sheets, SVGs, BOM
  and netlists. Labels are Confirmed / Likely / Unknown; Option A/B.
- netlist.py carries the ordering data of every BOM line: manufacturer,
  MPN, LCSC code with its evidence, JLCPCB class, price estimate, how it
  is assembled. bom.csv has the new columns; check.py rule R11 checks
  them and the selftest plants 12 faults.
- ORDERING.md: what to send a layout and assembly house, what is done
  and what the vendor does (the layout), the LT7911D documents to ask
  Lontium for, fabrication and assembly specs, bring-up tests, cost
  estimates at 10 and 50 boards, and an RFQ template.
- mechanical.py draws the enclosure outline and connector openings
  (svg/mechanical.svg).
- Design fixes: NRST note (4.7k), the end-of-life inductor replaced
  (SRP1038A-100M), the Bob-Smith capacitor rated 2 kV, capacitor ratings
  matched to stocked parts. Open points are listed in the README.

Co-Authored-By: Claude Opus 5.5 <noreply@anthropic.com>
Claude-Session: https://claude.ai/code/session_01EUDgAy5nU6wYzfaiaKBwjy
Parts:
- C301, C302: Confidence Chắc -> Confirmed; LCSC (none) -> C1549; MPN (none) -> 0402CG180J500NT; Manufacturer (none) -> FH (Guangdong Fenghua)
- C303, C304, C305, C306, C307, C308, C311: Confidence Chắc -> Confirmed; LCSC (none) -> C1525; MPN (none) -> CL05B104KO5NNNC; Manufacturer (none) -> Samsung Electro-Mechanics
- C309: value 1uF -> 1uF 25V; Confidence Chắc -> Confirmed; LCSC (none) -> C52923; MPN (none) -> CL05A105KA5NQNC; Manufacturer (none) -> Samsung Electro-Mechanics
- C310: value 10uF 6.3V -> 10uF 10V; Confidence Chắc -> Confirmed; LCSC (none) -> C19702; MPN (none) -> CL10A106KP8NNNC; Manufacturer (none) -> Samsung Electro-Mechanics
- C312, C313: Confidence Chắc -> Confirmed; LCSC (none) -> C1523; MPN (none) -> 0402B102K500NT; Manufacturer (none) -> FH (Guangdong Fenghua)
- C314: Confidence Chắc -> Confirmed; LCSC (none) -> C15195; MPN (none) -> CL05B103KB5NNNC; Manufacturer (none) -> Samsung Electro-Mechanics
- FB301: Confidence Chắc -> Confirmed; LCSC (none) -> C85833; Manufacturer (none) -> Murata
- R301: Confidence Chắc -> Confirmed; LCSC (none) -> C25900; MPN (none) -> 0402WGF4701TCE; Manufacturer (none) -> UNI-ROYAL (Uniroyal Elec)
- R302, R303: Confidence Chắc -> Confirmed; LCSC (none) -> C25744; MPN (none) -> 0402WGF1002TCE; Manufacturer (none) -> UNI-ROYAL (Uniroyal Elec)
- R304, R305, R306: Confidence Chắc -> Confirmed; LCSC (none) -> C25741; MPN (none) -> 0402WGF1003TCE; Manufacturer (none) -> UNI-ROYAL (Uniroyal Elec)
- R307: Confidence Chắc -> Confirmed; LCSC (none) -> C25756; MPN (none) -> 0402WGF1502TCE; Manufacturer (none) -> UNI-ROYAL (Uniroyal Elec)
- U301: Confidence Chắc -> Confirmed; Manufacturer (none) -> WCH (Jiangsu Qin Heng)
- X301: Confidence Chắc -> Confirmed; LCSC (none) -> C2682775; MPN (none) -> X32258MOB4SI; Manufacturer (none) -> YXC (Yangxing Tech)
Other:
- note added: "3. CH32V305RBT6: USB HS HID to the iPhone, SPI/UART link to the RV1106"
- note added: "Net labels sit on the pin ends (no wires). Pin numbers '?..' = no datasheet yet, must be confirmed before footprint/layout work."
- note removed: "3. CH32V305RBT6: USB HS HID tới iPhone, link SPI/UART tới RV1106"
- note removed: "Nhãn net đặt ngay đầu chân (không vẽ dây). Chân số '?..' = chưa có datasheet, phải xác nhận trước khi làm footprint/layout."
