File: hardware/box-v1/kicad/power.kicad_sch (KiCad schematic)
At the start: 78 parts, among them J101 USB-C PD IN, Q101 AO4407A, Q102 AO4407A, Q103 2N7002, U101 CH224K, U102 LMR33630ADDA, U103 LMR33630ADDA, U104 TLV62569DBV, U105 TLV62569DBV, U106 INA180A2

Commit message: hardware/box-v1 in English, with an order package
- Everything in hardware/box-v1 is English: netlist.py, the generators,
  the checks, the README, and the regenerated KiCad sheets, SVGs, BOM
  and netlists. Labels are Confirmed / Likely / Unknown; Option A/B.
- netlist.py carries the ordering data of every BOM line: manufacturer,
  MPN, LCSC code with its evidence, JLCPCB class, price estimate, how it
  is assembled. bom.csv has the new columns; check.py rule R11 checks
  them and the selftest plants 12 faults.
- ORDERING.md: what to send a layout and assembly house, what is done
  and what the vendor does (the layout), the LT7911D documents to ask
  Lontium for, fabrication and assembly specs, bring-up tests, cost
  estimates at 10 and 50 boards, and an RFQ template.
- mechanical.py draws the enclosure outline and connector openings
  (svg/mechanical.svg).
- Design fixes: NRST note (4.7k), the end-of-life inductor replaced
  (SRP1038A-100M), the Bob-Smith capacitor rated 2 kV, capacitor ratings
  matched to stocked parts. Open points are listed in the README.

Co-Authored-By: Claude Opus 5.5 <noreply@anthropic.com>
Claude-Session: https://claude.ai/code/session_01EUDgAy5nU6wYzfaiaKBwjy
Parts:
- C101: Confidence Chắc -> Confirmed; LCSC (none) -> C2836440; MPN nhôm polymer/điện phân 47 µF 35 V 6.3x7.7 -> RVT47UF35V67RV0039; Manufacturer (none) -> KNSCHA
- C102: value 1uF 25V -> 1uF 50V; Confidence Chắc -> Confirmed; LCSC (none) -> C15849; MPN (none) -> CL10A105KB8NNNC; Manufacturer (none) -> Samsung Electro-Mechanics
- C103, C104, C111, C112: Confidence Chắc -> Confirmed; LCSC (none) -> C89632; MPN (none) -> CL31B106KBHNNNE; Manufacturer (none) -> Samsung Electro-Mechanics
- C105, C113: Confidence Chắc -> Confirmed; LCSC (none) -> C14663; MPN (none) -> CC0603KRX7R9BB104; Manufacturer (none) -> YAGEO
- C106, C114: value 1uF 16V -> 1uF 25V; Confidence Chắc -> Confirmed; LCSC (none) -> C52923; MPN (none) -> CL05A105KA5NQNC; Manufacturer (none) -> Samsung Electro-Mechanics
- C107, C115, C120, C124, C125, C129: Confidence Chắc -> Confirmed; LCSC (none) -> C1525; MPN (none) -> CL05B104KO5NNNC; Manufacturer (none) -> Samsung Electro-Mechanics
- C108, C109, C110, C116, C117, C118: value 22uF 10V X5R -> 22uF 25V X5R; Confidence Chắc -> Confirmed; LCSC (none) -> C12891; MPN (none) -> CL31A226KAHNNNE; Manufacturer (none) -> Samsung Electro-Mechanics
- C119, C123: Confidence Chắc -> Confirmed; LCSC (none) -> C19702; MPN (none) -> CL10A106KP8NNNC; Manufacturer (none) -> Samsung Electro-Mechanics
- C121, C122, C126, C127: value 22uF 6.3V X5R -> 22uF 25V X5R; Confidence Chắc -> Confirmed; LCSC (none) -> C45783; MPN (none) -> CL21A226MAQNNNE; Manufacturer (none) -> Samsung Electro-Mechanics
- C128: footprint Capacitor_SMD:C_0402_1005Metric -> Capacitor_SMD:C_0603_1608Metric; Confidence Chắc -> Confirmed; LCSC (none) -> C1622; MPN (none) -> CL10B473KB8NNNC; Manufacturer (none) -> Samsung Electro-Mechanics
- C130: Confidence Chắc -> Confirmed; LCSC (none) -> C1523; MPN (none) -> 0402B102K500NT; Manufacturer (none) -> FH (Guangdong Fenghua)
- D101: Confidence Chắc -> Confirmed; LCSC (none) -> C19077541; Manufacturer (none) -> hongjiacheng
- D102: Confidence Chắc -> Confirmed; LCSC (none) -> C155227; MPN BZT52C10 -> BZT52C10-7-F; Manufacturer (none) -> Diodes Incorporated
- D104: Confidence Chắc -> Confirmed; LCSC (none) -> C8678; Manufacturer (none) -> MDD (Microdiode Electronics)
- F101: Confidence Có thể -> Likely; LCSC (none) -> C57525; MPN Littelfuse 0466005.NR -> 0466005.NRHF; Manufacturer (none) -> Littelfuse
- J101: Confidence Chắc -> Confirmed; Manufacturer (none) -> Korean Hroparts Elec; Note D+/D- để trống: CH224K chạy chế độ chỉ PD (datasheet CH224 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 -> D+/D- left open: the CH224K runs in PD-only mode (CH224 dat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
- JP101: Confidence Chắc -> Confirmed; MPN (none) -> none (solder jumper on the PCB); Manufacturer (none) -> -; Note Làm pad rộng ≥ 2 mm, phủ thiếc dày: dòng 3 A -> Make the pads ≥ 2 mm wide with a thick solder coat: 3 A
- JP102: Confidence Chắc -> Confirmed; MPN (none) -> none (solder jumper on the PCB); Manufacturer (none) -> -
- L101, L102: Confidence Có thể -> Likely; LCSC (none) -> C780184; MPN Bourns SRP1038C-100M (hoặc tương đương) -> SRP1038A-100M; Manufacturer (none) -> Bourns
- L103, L104: Confidence Có thể -> Likely; LCSC (none) -> C913207; MPN Bourns SRN4018-2R2M (hoặc tương đương) -> SRN4018-2R2M; Manufacturer (none) -> Bourns
- Q101, Q102: Confidence Có thể -> Likely; LCSC (none) -> C16072; Manufacturer (none) -> Alpha & Omega Semiconductor; Note Sơ đồ chân SO-8 MOSFET chuẩn (S=1-3, G=4, D=5-8), như ký hi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 -> Standard SO-8 MOSFET pinout (S=1-3, G=4, D=5-8), as the KiC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
- Q103: Confidence Chắc -> Confirmed; LCSC (none) -> C8545; Manufacturer (none) -> Changjiang Electronics Tech (CJ)
- R101: Confidence Chắc -> Confirmed; LCSC (none) -> C4410; MPN (none) -> 1206W4F1001T5E; Manufacturer (none) -> UNI-ROYAL (Uniroyal Elec); Note 1206 (0.25 W): ở 15 V tiêu tán 0.14 W -> 1206 (0.25 W): dissipates 0.14 W at 15 V
- R102, R108, R124: Confidence Chắc -> Confirmed; LCSC (none) -> C25744; MPN (none) -> 0402WGF1002TCE; Manufacturer (none) -> UNI-ROYAL (Uniroyal Elec)
- R103: Confidence Chắc -> Confirmed; LCSC (none) -> C25917; MPN (none) -> 0402WGF6801TCE; Manufacturer (none) -> UNI-ROYAL (Uniroyal Elec)
- R104, R105, R127: Confidence Chắc -> Confirmed; LCSC (none) -> C17168; MPN (none) -> 0402WGF0000TCE; Manufacturer (none) -> UNI-ROYAL (Uniroyal Elec)
- R106, R107, R128: Confidence Chưa biết -> Unknown; LCSC (none) -> C17168; MPN (none) -> 0402WGF0000TCE; Manufacturer (none) -> UNI-ROYAL (Uniroyal Elec)
- R109, R111, R113, R115, R117, R118, R120, R121, R122, R123, R125: Confidence Chắc -> Confirmed; LCSC (none) -> C25741; MPN (none) -> 0402WGF1003TCE; Manufacturer (none) -> UNI-ROYAL (Uniroyal Elec)
- R110: Confidence Chắc -> Confirmed; LCSC (none) -> C327362; MPN (none) -> RC0402FR-0723K7L; Manufacturer (none) -> YAGEO
- R112: Confidence Chắc -> Confirmed; LCSC (none) -> C25765; MPN (none) -> 0402WGF2002TCE; Manufacturer (none) -> UNI-ROYAL (Uniroyal Elec)
- R114: Confidence Chắc -> Confirmed; MPN (none) -> RC0402FR-0724K9L; Manufacturer (none) -> YAGEO
- R116: Confidence Chắc -> Confirmed; LCSC (none) -> C25783; MPN (none) -> 0402WGF3902TCE; Manufacturer (none) -> UNI-ROYAL (Uniroyal Elec)
- R119: Confidence Chắc -> Confirmed; MPN (none) -> RC0402FR-0722K1L; Manufacturer (none) -> YAGEO
- R126: Confidence Chắc -> Confirmed; LCSC (none) -> C155193; MPN 1206 10 mΩ 1% 0.5 W -> RL1206FR-7W0R01L; Manufacturer (none) -> YAGEO
- U101: Confidence Chắc -> Confirmed; Manufacturer (none) -> WCH (Jiangsu Qin Heng)
- U102, U103: Confidence Có thể -> Likely; Manufacturer (none) -> Texas Instruments; Note VREF 1.0 V, ngưỡng EN ~1.2 V: đọc lại datasheet TI SNVSAX4 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 -> VREF 1.0 V, EN threshold ~1.2 V: re-read TI datasheet SNVSA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
- U104, U105: Confidence Có thể -> Likely; LCSC (none) -> C141836; Manufacturer (none) -> Texas Instruments; Note VREF 0.6 V, 1.5 MHz: đọc lại datasheet TI SLVSDI0 -> VREF 0.6 V, 1.5 MHz: re-read TI datasheet SLVSDI0
- U106: Confidence Có thể -> Likely; LCSC (none) -> C192764; Manufacturer (none) -> Texas Instruments
Other:
- note added: "1. Power: USB-C PD input (CH224K), 5V2/5V/3V3/1V2 bucks, iPhone VBUS switch"
- note added: "Net labels sit on the pin ends (no wires). Pin numbers '?..' = no datasheet yet, must be confirmed before footprint/layout work."
- note added: "PWR_FLAG (ERC): rails fed through an inductor/resistor/connector"
- note removed: "1. Nguồn: USB-C PD vào (CH224K), buck 5V2/5V/3V3/1V2, công tắc VBUS iPhone"
- note removed: "Nhãn net đặt ngay đầu chân (không vẽ dây). Chân số '?..' = chưa có datasheet, phải xác nhận trước khi làm footprint/layout."
- note removed: "PWR_FLAG (ERC): rail được cấp qua cuộn cảm/điện trở/đầu nối"
- title: box-v1: nguồn -> box-v1: power

Commit message: Box v1: second design review and a PCB generator
- netlist.py: CH224K VBUS pin left open (R102 removed); D101 SMBJ20A clamps
  below the LMR33630's 36 V input; U107 ESD on the rear CC lines; R213 and a
  100 nF C215 on the LT7911D reset; I2C pull-ups on the module's 3.3 V; J201
  HRO TYPE-C-31-M-04 (hybrid, routable B row); TS-1187A buttons; net classes
  shared with the project file and the board.
- placement.py, pcb.py: the 96x66 mm 4-layer board generated from the
  netlist: footprints (custom LT7911D, Core1106, CH224K, vendored HRO
  receptacle), placement, rules, keep-outs, GND fan-out and stitching,
  Freerouting 1.9 round trip, zones, DRC, compact SVG views.
- mechanical.py follows placement.py; README §11, §14, §15 and ORDERING.md
  describe the layout, the review and the remaining LT7911D work; the
  LT7911D datasheet is public on LCSC.

Co-Authored-By: Claude Opus 5.5 <noreply@anthropic.com>
Claude-Session: https://claude.ai/code/session_01EUDgAy5nU6wYzfaiaKBwjy
Parts:
- removed R102: 10k, Resistor_SMD:R_0402_1005Metric, symbol box-v1:R
- added U107: TPD4E05U06DQA, Package_SON:USON-10_2.5x1.0mm_P0.5mm, symbol box-v1:TPD4E05U06DQA_dd89b8
- D101: value SMAJ24A -> SMBJ20A; footprint Diode_SMD:D_SMA -> Diode_SMD:D_SMB; LCSC C19077541 -> C19077575; MPN SMAJ24A -> SMBJ20A
- R101: Note 1206 (0.25 W): dissipates 0.14 W at 15 V -> 1206 (0.25 W): 0.14 W at 15 V; a 20 V request (R103 open) w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
Connections:
- net GND: now also U107.3 (GND), U107.8 (GND)
- net PD_CC1: now also U107.1 (D1+)
- net PD_CC2: now also U107.2 (D1-)
- net CH224_VSNS: no longer names the net of U101.8 (VBUS)
- new net PC_CC1: U107.4 (D2+)
- new net PC_CC2: U107.5 (D2-)
- no-connect marks 10 -> 15
Other:
- moved on the sheet: C103, C104, C105, C106, C107, C108, C109, C110, C111, C112, C113, C114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
