File: hardware/box-v1/kicad/soc.kicad_sch (KiCad schematic)
At the start: 29 parts, among them J401 USB-C PC, J402 RJ45 10/100, U401 Luckfox Core1106, U402 USBLC6-2SC6

Commit message: hardware/box-v1 in English, with an order package
- Everything in hardware/box-v1 is English: netlist.py, the generators,
  the checks, the README, and the regenerated KiCad sheets, SVGs, BOM
  and netlists. Labels are Confirmed / Likely / Unknown; Option A/B.
- netlist.py carries the ordering data of every BOM line: manufacturer,
  MPN, LCSC code with its evidence, JLCPCB class, price estimate, how it
  is assembled. bom.csv has the new columns; check.py rule R11 checks
  them and the selftest plants 12 faults.
- ORDERING.md: what to send a layout and assembly house, what is done
  and what the vendor does (the layout), the LT7911D documents to ask
  Lontium for, fabrication and assembly specs, bring-up tests, cost
  estimates at 10 and 50 boards, and an RFQ template.
- mechanical.py draws the enclosure outline and connector openings
  (svg/mechanical.svg).
- Design fixes: NRST note (4.7k), the end-of-life inductor replaced
  (SRP1038A-100M), the Bob-Smith capacitor rated 2 kV, capacitor ratings
  matched to stocked parts. Open points are listed in the README.

Co-Authored-By: Claude Opus 5.5 <noreply@anthropic.com>
Claude-Session: https://claude.ai/code/session_01EUDgAy5nU6wYzfaiaKBwjy
Parts:
- C401: value 22uF 10V -> 22uF 25V X5R; Confidence Chắc -> Confirmed; LCSC (none) -> C45783; MPN (none) -> CL21A226MAQNNNE; Manufacturer (none) -> Samsung Electro-Mechanics
- C402, C403, C405: Confidence Chắc -> Confirmed; LCSC (none) -> C1525; MPN (none) -> CL05B104KO5NNNC; Manufacturer (none) -> Samsung Electro-Mechanics
- C404: value 1uF 25V -> 1uF 50V; Confidence Chắc -> Confirmed; LCSC (none) -> C15849; MPN (none) -> CL10A105KB8NNNC; Manufacturer (none) -> Samsung Electro-Mechanics
- C406, C407, C409: Confidence Chắc -> Confirmed; LCSC (none) -> C15195; MPN (none) -> CL05B103KB5NNNC; Manufacturer (none) -> Samsung Electro-Mechanics
- C408: value 1nF 100V -> 1nF 2kV X7R; footprint Capacitor_SMD:C_0603_1608Metric -> Capacitor_SMD:C_1206_3216Metric; Confidence Chắc -> Confirmed; LCSC (none) -> C9196; MPN (none) -> 1206B102K202NT; Manufacturer (none) -> FH (Guangdong Fenghua)
- C410: Confidence Chắc -> Confirmed; LCSC (none) -> C76947; MPN (none) -> GRM1555C1H102JA01D; Manufacturer (none) -> Murata
- D401: Confidence Chắc -> Confirmed; LCSC (none) -> C207260; Manufacturer (none) -> Littelfuse
- J401: Confidence Chắc -> Confirmed; Manufacturer (none) -> Korean Hroparts Elec
- J402: Confidence Chắc -> Confirmed; Manufacturer (none) -> HANRUN (Zhongshan HanRun Elec)
- R401, R402: Confidence Chắc -> Confirmed; LCSC (none) -> C25905; MPN (none) -> 0402WGF5101TCE; Manufacturer (none) -> UNI-ROYAL (Uniroyal Elec)
- R403, R411: Confidence Chắc -> Confirmed; LCSC (none) -> C25744; MPN (none) -> 0402WGF1002TCE; Manufacturer (none) -> UNI-ROYAL (Uniroyal Elec)
- R404: Confidence Chắc -> Confirmed; LCSC (none) -> C25762; MPN (none) -> 0402WGF1802TCE; Manufacturer (none) -> UNI-ROYAL (Uniroyal Elec)
- R405, R406, R407, R408: Confidence Chắc -> Confirmed; LCSC (none) -> C17168; MPN (none) -> 0402WGF0000TCE; Manufacturer (none) -> UNI-ROYAL (Uniroyal Elec)
- R409: Confidence Chắc -> Confirmed; LCSC (none) -> C25741; MPN (none) -> 0402WGF1003TCE; Manufacturer (none) -> UNI-ROYAL (Uniroyal Elec)
- R410: Confidence Chắc -> Confirmed; LCSC (none) -> C25924; MPN (none) -> 0402WGF8201TCE; Manufacturer (none) -> UNI-ROYAL (Uniroyal Elec)
- R412: Confidence Chắc -> Confirmed; LCSC (none) -> C25076; MPN (none) -> 0402WGF1000TCE; Manufacturer (none) -> UNI-ROYAL (Uniroyal Elec)
- R413: Confidence Chắc -> Confirmed; LCSC (none) -> C11702; MPN (none) -> 0402WGF1001TCE; Manufacturer (none) -> UNI-ROYAL (Uniroyal Elec)
- TP401: Confidence Chắc -> Confirmed; MPN (none) -> none (copper test pad); Manufacturer (none) -> -
- U401: Confidence Có thể -> Likely; MPN Luckfox Core1106 (RV1106G3, 256 MB, eMMC 8 GB, Wi-Fi 6/BT 5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 -> Core1106 (RV1106G3, 256 MB, 8 GB eMMC, Wi-Fi 6/BT 5.2 varia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; Manufacturer (none) -> Luckfox; Note Footprint: dùng Core1106-SMT của Luckfox (30x30 mm, 112 pad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 -> Footprint: use Luckfox Core1106-SMT (30x30 mm, 112 pads, 1.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
- U402: Confidence Chắc -> Confirmed; Manufacturer (none) -> STMicroelectronics
Other:
- note added: "4. Luckfox Core1106 (RV1106G3) + 100M RJ45 + USB-C to the PC"
- note added: "Net labels sit on the pin ends (no wires). Pin numbers '?..' = no datasheet yet, must be confirmed before footprint/layout work."
- note removed: "4. Luckfox Core1106 (RV1106G3) + RJ45 100M + USB-C tới PC"
- note removed: "Nhãn net đặt ngay đầu chân (không vẽ dây). Chân số '?..' = chưa có datasheet, phải xác nhận trước khi làm footprint/layout."
- title: box-v1: Core1106 + Ethernet + USB PC -> box-v1: Core1106 + Ethernet + PC USB

Commit message: Box v1: second design review and a PCB generator
- netlist.py: CH224K VBUS pin left open (R102 removed); D101 SMBJ20A clamps
  below the LMR33630's 36 V input; U107 ESD on the rear CC lines; R213 and a
  100 nF C215 on the LT7911D reset; I2C pull-ups on the module's 3.3 V; J201
  HRO TYPE-C-31-M-04 (hybrid, routable B row); TS-1187A buttons; net classes
  shared with the project file and the board.
- placement.py, pcb.py: the 96x66 mm 4-layer board generated from the
  netlist: footprints (custom LT7911D, Core1106, CH224K, vendored HRO
  receptacle), placement, rules, keep-outs, GND fan-out and stitching,
  Freerouting 1.9 round trip, zones, DRC, compact SVG views.
- mechanical.py follows placement.py; README §11, §14, §15 and ORDERING.md
  describe the layout, the review and the remaining LT7911D work; the
  LT7911D datasheet is public on LCSC.

Co-Authored-By: Claude Opus 5.5 <noreply@anthropic.com>
Claude-Session: https://claude.ai/code/session_01EUDgAy5nU6wYzfaiaKBwjy
Connections:
- net LT_RST_N renamed SOC_LT_RST
